File: BBLEDTemplate.sch (KiCad schematic (older format))
At the start: 11 parts

Commit message: add values
Parts:
- C? (x4): value C0603 -> 0.1u
Changed lines of the file:
@@
 P 4350 4200
 F 0 "C?" H 4465 4246 50  0000 L CNN
-F 1 "C0603" H 4465 4155 50  0000 L CNN
+F 1 "0.1u" H 4465 4155 50  0000 L CNN
 F 2 "Capacitor_SMD:C_0603_1608Metric" H 4388 4050 50  0001 C CNN
 F 3 "" H 4350 4200 50  0001 C CNN
@@
 P 4950 4200
 F 0 "C?" H 5065 4246 50  0000 L CNN
-F 1 "C0603" H 5065 4155 50  0000 L CNN
+F 1 "0.1u" H 5065 4155 50  0000 L CNN
 F 2 "Capacitor_SMD:C_0603_1608Metric" H 4988 4050 50  0001 C CNN
 F 3 "" H 4950 4200 50  0001 C CNN
@@
 P 5550 4200
 F 0 "C?" H 5665 4246 50  0000 L CNN
-F 1 "C0603" H 5665 4155 50  0000 L CNN
+F 1 "0.1u" H 5665 4155 50  0000 L CNN
 F 2 "Capacitor_SMD:C_0603_1608Metric" H 5588 4050 50  0001 C CNN
 F 3 "" H 5550 4200 50  0001 C CNN
@@
 P 6150 4200
 F 0 "C?" H 6265 4246 50  0000 L CNN
-F 1 "C0603" H 6265 4155 50  0000 L CNN
+F 1 "0.1u" H 6265 4155 50  0000 L CNN
 F 2 "Capacitor_SMD:C_0603_1608Metric" H 6188 4050 50  0001 C CNN
 F 3 "" H 6150 4200 50  0001 C CNN
